Commit message: Stability and performance fix, added toggling between gazebo & ros2_control

File: description/robot.urdf.xacro (robot description, xacro)
@@ -1,7 +1,12 @@
 <?xml version="1.0"?>
 <robot xmlns:xacro="http://www.ros.org/wiki/xacro"  name="robot">
+    <xacro:arg name="use_ros2_control" default="true"/>
     <xacro:include filename="robot_core.xacro" />
-    <!-- <xacro:include filename="gazebo_control.xacro"/> -->
-    <xacro:include filename="ros2_control.xacro"/>
+    <xacro:if value="$(arg use_ros2_control)">
+        <xacro:include filename="ros2_control.xacro" />
+    </xacro:if>
+    <xacro:unless value="$(arg use_ros2_control)">
+        <xacro:include filename="gazebo_control.xacro" />
+    </xacro:unless>
     <xacro:include filename="lidar.xacro"/>
     <!-- <xacro:include filename="camera.xacro"/> -->

File: description/robot_core.xacro (robot description, xacro)
@@ -50,4 +50,6 @@
     </joint>
     <!-- Design of wheels at your discretion -->
+    <!-- To avoid wheel drift in simulation (causing odom desync between Gazebo and RViz), have collision geometry to be a Sphere instead,
+        reduces the contact point to be infinitely small -->
     <link name="left_wheel">
         <visual>
@@ -59,5 +61,6 @@
         <collision>
             <geometry>
-                <cylinder length="0.04" radius="0.05"/>
+                <!-- <cylinder length="0.04" radius="0.05"/> -->
+                <sphere radius="0.05"/>
             </geometry>
         </collision>
@@ -76,4 +79,6 @@
     </joint>
     <!-- Design of wheels at your discretion -->
+    <!-- To avoid wheel drift in simulation (causing odom desync between Gazebo and RViz), have collision geometry to be a Sphere instead,
+        reduces the contact point to be infinitely small -->
     <link name="right_wheel">
         <visual>
@@ -85,5 +90,6 @@
         <collision>
             <geometry>
-                <cylinder length="0.04" radius="0.05"/>
+                <!-- <cylinder length="0.04" radius="0.05"/> -->
+                <sphere radius="0.05"/>
             </geometry>
         </collision>
