Commit message: Driving with DiffDrive plugin

File: description/robot_core.xacro (robot description, xacro)
@@ -36,4 +36,8 @@
         </xacro:inertial_box>
     </link>
+    <!-- Should Gazebo be mising colors, add the following lines under each link tag -->
+    <!-- <gazebo reference="chassis">
+        <material>Gazebo/White</material>
+    </gazebo> -->
     <!-- LEFT WHEEL LINK -->
     <!-- Origin refer to mock-up design -->
@@ -112,3 +116,8 @@
         </xacro:inertial_sphere>
     </link>
+    <!-- Configure friction coefficients mu1 and mu2, set to either zero or small number at your choosing -->
+    <gazebo reference="caster_wheel">
+        <mu1 value="0.001"/>
+        <mu2 value="0.001"/>
+    </gazebo>
 </robot>

Commit message: Added SLAM-based mapping

File: description/robot_core.xacro (robot description, xacro)
@@ -6,4 +6,13 @@
     <!-- Treating center of the two drive wheels as the origin (for DiffDrive robot) -->
     <link name="base_link">
+    </link>
+    <!-- BASE_FOOTPRINT LINK -->
+    <!-- created just for SLAM, acts as a shadow of base_link on the ground, constrain within x-y plane -->
+    <joint name="base_footprint_joint" type="fixed">
+        <parent link="base_link"/>
+        <child link="base_footprint"/>
+        <origin xyz="0 0 0" rpy="0 0 0"/>
+    </joint>
+    <link name="base_footprint">
     </link>
     <!-- CHASSIS LINK -->
